Commit message: added controllers to project

File: urdf/car.xacro (robot description, xacro)
@@ -971,3 +971,177 @@
       xyz="-0.00252374300930457 0 -0.99999681535554" />
   </joint>
+  <ros2_control name="GazeboSystem" type="system">
+    <hardware>
+        <plugin>gazebo_ros2_control/GazeboSystem</plugin>
+    </hardware>
+    # Velocity Controllers for 2 back wheels
+    <joint name="front_left_wheel_joint">
+      <command_interface name="velocity">
+          <param name="min">-1000.0</param>
+          <param name="max">1000.0</param>
+      </command_interface>
+      <state_interface name="position"/>
+      <state_interface name="velocity"/>
+  </joint>
+  <joint name="front_right_wheel_joint">
+    <command_interface name="velocity">
+        <param name="min">-1000.0</param>
+        <param name="max">1000.0</param>
+    </command_interface>
+    <state_interface name="position"/>
+    <state_interface name="velocity"/>
+  </joint>
+    <joint name="back_left_wheel_joint">
+        <command_interface name="velocity">
+            <param name="min">-1000.0</param>
+            <param name="max">1000.0</param>
+        </command_interface>
+        <state_interface name="position"/>
+        <state_interface name="velocity"/>
+    </joint>
+    <joint name="back_right_wheel_link_joint">
+      <command_interface name="velocity">
+          <param name="min">-1000.0</param>
+          <param name="max">1000.0</param>
+      </command_interface>
+      <state_interface name="position"/>
+      <state_interface name="velocity"/>
+  </joint>
+  <!-- Velocity controllers for ur10 -->
+  <joint name="01j">
+    <command_interface name="velocity">
+        <param name="min">-1000.0</param>
+        <param name="max">1000.0</param>
+    </command_interface>
+    <state_interface name="position"/>
+    <state_interface name="velocity"/>
+</joint>
+<joint name="12j">
+  <command_interface name="velocity">
+      <param name="min">-1000.0</param>
+      <param name="max">1000.0</param>
+  </command_interface>
+  <state_interface name="position"/>
+  <state_interface name="velocity"/>
+</joint>
+<joint name="23j">
+  <command_interface name="velocity">
+      <param name="min">-1000.0</param>
+      <param name="max">1000.0</param>
+  </command_interface>
+  <state_interface name="position"/>
+  <state_interface name="velocity"/>
+</joint>
+<joint name="34j">
+  <command_interface name="velocity">
+      <param name="min">-1000.0</param>
+      <param name="max">1000.0</param>
+  </command_interface>
+  <state_interface name="position"/>
+  <state_interface name="velocity"/>
+</joint>
+<joint name="45j">
+  <command_interface name="velocity">
+      <param name="min">-1000.0</param>
+      <param name="max">1000.0</param>
+  </command_interface>
+  <state_interface name="position"/>
+  <state_interface name="velocity"/>
+</joint>
+<joint name="56j">
+  <command_interface name="velocity">
+      <param name="min">-1000.0</param>
+      <param name="max">1000.0</param>
+  </command_interface>
+  <state_interface name="position"/>
+  <state_interface name="velocity"/>
+</joint>
+<joint name="67j">
+  <command_interface name="velocity">
+      <param name="min">-1000.0</param>
+      <param name="max">1000.0</param>
+  </command_interface>
+  <state_interface name="position"/>
+  <state_interface name="velocity"/>
+</joint>
+   # Position Controller for 2 front wheels
+    <joint name="front_right_link_joint">
+        <command_interface name="position">
+            <param name="min">-3.14</param>
+            <param name="max">3.14</param>
+        </command_interface>
+        <state_interface name="position"/>
+        <state_interface name="velocity"/>
+    </joint>
+    <joint name="front_left_link_joint">
+      <command_interface name="position">
+          <param name="min">-3.14</param>
+          <param name="max">3.14</param>
+      </command_interface>
+      <state_interface name="position"/>
+      <state_interface name="velocity"/>
+  </joint>
+  <!-- postion control for UR10 arms -->
+  <joint name="01j">
+    <command_interface name="position">
+        <param name="min">-3.14</param>
+        <param name="max">3.14</param>
+    </command_interface>
+    <state_interface name="position"/>
+    <state_interface name="velocity"/>
+</joint>
+<joint name="12j">
+  <command_interface name="position">
+      <param name="min">-3.14</param>
+      <param name="max">3.14</param>
+  </command_interface>
+  <state_interface name="position"/>
+  <state_interface name="velocity"/>
+</joint>
+<joint name="23j">
+  <command_interface name="position">
+      <param name="min">-3.14</param>
+      <param name="max">3.14</param>
+  </command_interface>
+  <state_interface name="position"/>
+  <state_interface name="velocity"/>
+</joint>
+<joint name="34j">
+  <command_interface name="position">
+      <param name="min">-3.14</param>
+      <param name="max">3.14</param>
+  </command_interface>
+  <state_interface name="position"/>
+  <state_interface name="velocity"/>
+</joint>
+<joint name="45j">
+  <command_interface name="position">
+      <param name="min">-3.14</param>
+      <param name="max">3.14</param>
+  </command_interface>
+  <state_interface name="position"/>
+  <state_interface name="velocity"/>
+</joint>
+<joint name="56j">
+  <command_interface name="position">
+      <param name="min">-3.14</param>
+      <param name="max">3.14</param>
+  </command_interface>
+  <state_interface name="position"/>
+  <state_interface name="velocity"/>
+</joint>
+<joint name="67j">
+  <command_interface name="position">
+      <param name="min">-3.14</param>
+      <param name="max">3.14</param>
+  </command_interface>
+  <state_interface name="position"/>
+  <state_interface name="velocity"/>
+</joint>
+    </ros2_control>
+    <gazebo>
+      <plugin filename="libgazebo_ros2_control.so" name="gazebo_ros2_control">
+          <parameters>$(find car)/config/control.yaml</parameters>
+      </plugin>
+  </gazebo>
 </robot>

Commit message: rviz spawn

File: urdf/car.xacro (robot description, xacro)
@@ -5,4 +5,10 @@
 <robot
   name="car" xmlns:xacro="http://ros.org/wiki/xacro">
+<link name="dummy_link"></link>
+<joint name="dummy_joint" type="fixed">
+    <origin rpy="0 0 0" xyz="0 0 0" />
+    <parent link="dummy_link"/>
+    <child link="car_base"/>
+</joint>
   <link
     name="car_base">

Commit message: new urdf with gripper

File: urdf/car.xacro (robot description, xacro)
@@ -3,17 +3,17 @@
      Commit Version: 1.6.0-4-g7f85cfe  Build Version: 1.6.7995.38578
      For more information, please see http://wiki.ros.org/sw_urdf_exporter -->
-<robot
-  name="car" xmlns:xacro="http://ros.org/wiki/xacro">
-<link name="dummy_link"></link>
-<joint name="dummy_joint" type="fixed">
-    <origin rpy="0 0 0" xyz="0 0 0" />
-    <parent link="dummy_link"/>
-    <child link="car_base"/>
-</joint>
+     <robot
+     name="car" xmlns:xacro="http://ros.org/wiki/xacro">
+   <link name="dummy_link"></link>
+   <joint name="dummy_joint" type="fixed">
+       <origin rpy="0 0 0" xyz="0 0 0" />
+       <parent link="dummy_link"/>
+       <child link="car_base"/>
+   </joint>
   <link
     name="car_base">
     <inertial>
       <origin
-        xyz="8.17360748943693E-06 0.0225033135182252 0.309234562686189"
+        xyz="8.17360748943708E-06 0.0225033135182252 0.309234562686189"
         rpy="0 0 0" />
       <mass
@@ -21,8 +21,8 @@
       <inertia
         ixx="64.8069935901443"
-        ixy="0.00212233959160385"
-        ixz="0.000377899491888436"
+        ixy="0.00212233959160378"
+        ixz="0.000377899491888311"
         iyy="42.2474032259228"
-        iyz="-1.35082963675343"
+        iyz="-1.35082963675344"
         izz="71.07249676203" />
     </inertial>
@@ -542,5 +542,5 @@
   <joint
     name="lidar_joint"
-    type="fixed">
+    type="continuous">
     <origin
       xyz="0 0.1524 0.655447"
@@ -551,5 +551,5 @@
       link="lidar_link" />
     <axis
-      xyz="0 0 0" />
+      xyz="0 0 1" />
   </joint>
   <link
@@ -557,5 +557,5 @@
     <inertial>
       <origin
-        xyz="7.22391839389283E-06 -0.000475137384490065 0.000654978643972126"
+        xyz="7.22391839388936E-06 -0.000475137384490038 0.000654978643972126"
         rpy="0 0 0" />
       <mass
@@ -563,8 +563,8 @@
       <inertia
         ixx="0.00312084570629235"
-        ixy="1.03835097415574E-07"
-        ixz="2.20016415043755E-07"
+        ixy="1.03835097415563E-07"
+        ixz="2.20016415043754E-07"
         iyy="0.00309492725703448"
-        iyz="5.55031448922638E-07"
+        iyz="5.55031448922626E-07"
         izz="0.00574920281992534" />
     </inertial>
@@ -610,12 +610,12 @@
     <inertial>
       <origin
-        xyz="3.70762208490583E-05 0.0114409852434528 0.0116125856420283"
-        rpy="0 0 0" />
-      <mass
-        value="8.30725875791485" />
+        xyz="3.70762208490617E-05 0.0114409852434533 0.0116125856420283"
+        rpy="0 0 0" />
+      <mass
+        value="8.30725875791486" />
       <inertia
         ixx="0.029020927491474"
-        ixy="7.55948089001624E-06"
-        ixz="-8.23045819536526E-06"
+        ixy="7.55948089001623E-06"
+        ixz="-8.23045819536529E-06"
         iyy="0.027224956518295"
         iyz="0.00281819311295836"
@@ -669,6 +669,6 @@
       <inertia
         ixx="0.256767671623099"
-        ixy="3.62399517884548E-06"
-        ixz="-9.72858775406835E-07"
+        ixy="3.6239951788455E-06"
+        ixz="-9.72858775406846E-07"
         iyy="0.0505710283974333"
         iyz="0.00203684454830707"
@@ -716,5 +716,5 @@
     <inertial>
       <origin
-        xyz="0.244390991313134 -0.0139095256822837 -0.00101283060327784"
+        xyz="0.244390991313135 -0.0139095256822837 -0.00101283060327786"
         rpy="0 0 0" />
       <mass
@@ -725,5 +725,5 @@
         ixz="-0.00028822454084213"
         iyy="0.131613662619847"
-        iyz="3.49342881189503E-07"
+        iyz="3.49342881189501E-07"
         izz="0.131781826183782" />
     </inertial>
@@ -775,9 +775,9 @@
       <inertia
         ixx="0.000910114210779735"
-        ixy="-4.95497562223857E-07"
+        ixy="-4.95497562223844E-07"
         ixz="-0.00012008521723334"
-        iyy="0.000986687923606721"
-        iyz="-1.62299300727914E-07"
-        izz="0.000877255272961633" />
+        iyy="0.000986687923606722"
+        iyz="-1.62299300727913E-07"
+        izz="0.000877255272961634" />
     </inertial>
     <visual>
@@ -822,5 +822,5 @@
     <inertial>
       <origin
-        xyz="-6.86078064258272E-06 -0.00758686562123934 0.0107376301790447"
+        xyz="-6.86078064257925E-06 -0.00758686562123945 0.0107376301790445"
         rpy="0 0 0" />
       <mass
@@ -828,6 +828,6 @@
       <inertia
         ixx="0.000986687619429261"
-        ixy="-1.03152618194114E-09"
-        ixz="-4.17354729205834E-07"
+        ixy="-1.0315261819144E-09"
+        ixz="-4.1735472920583E-07"
         iyy="0.000910112478523473"
         iyz="-0.000120085251276709"
@@ -880,10 +880,10 @@
         value="0.728997478631908" />
       <inertia
-        ixx="0.00098668725075459"
-        ixy="4.95491590353946E-07"
-        ixz="-1.62291043906277E-07"
+        ixx="0.000986687250754589"
+        ixy="4.95491590354025E-07"
+        ixz="-1.62291043906281E-07"
         iyy="0.000910112496687827"
         iyz="0.000120084923500319"
-        izz="0.000877253430656249" />
+        izz="0.000877253430656248" />
     </inertial>
     <visual>
@@ -928,5 +928,5 @@
     <inertial>
       <origin
-        xyz="-5.11211491377381E-05 -0.000470150585815121 -0.00309378276926547"
+        xyz="-5.11211491377381E-05 -0.000470150585815121 -0.00309378276926542"
         rpy="0 0 0" />
       <mass
@@ -976,4 +976,57 @@
     <axis
       xyz="-0.00252374300930457 0 -0.99999681535554" />
+  </joint>
+  <link
+    name="gripper">
+    <inertial>
+      <origin
+        xyz="-0.00710247160346223 0.0303390950483817 0.000488474590246035"
+        rpy="0 0 0" />
+      <mass
+        value="1.34963431952749" />
+      <inertia
+        ixx="0.00651208089817064"
+        ixy="0.000182430404454022"
+        ixz="-0.000121865713788611"
+        iyy="0.00861283977900374"
+        iyz="-1.31090652690096E-05"
+        izz="0.0049440363866004" />
+    </inertial>
+    <visual>
+      <origin
+        xyz="0 0 0"
+        rpy="0 0 0" />
+      <geometry>
+        <mesh
+          filename="package://car/meshes/gripper.STL" />
+      </geometry>
+      <material
+        name="">
+        <color
+          rgba="0.2 0.2 0.2 1" />
+      </material>
+    </visual>
+    <collision>
+      <origin
+        xyz="0 0 0"
+        rpy="0 0 0" />
+      <geometry>
+        <mesh
+          filename="package://car/meshes/gripper.STL" />
+      </geometry>
+    </collision>
+  </link>
+  <joint
+    name="7-gripper_joint"
+    type="fixed">
+    <origin
+      xyz="-0.000514480216416438 0.000109109397764318 0.0968676227049757"
+      rpy="-1.5707963267949 0 3.14159265358979" />
+    <parent
+      link="67" />
+    <child
+      link="gripper" />
+    <axis
+      xyz="0 0 0" />
   </joint>
   <ros2_control name="GazeboSystem" type="system">

Commit message: circle trajectory node urdf changed with coorect axis updated dh table

File: urdf/car.xacro (robot description, xacro)
@@ -15,5 +15,5 @@
     <inertial>
       <origin
-        xyz="8.17360748943708E-06 0.0225033135182252 0.309234562686189"
+        xyz="8.17360748944015E-06 0.0225033135182252 0.309234562686189"
         rpy="0 0 0" />
       <mass
@@ -21,6 +21,6 @@
       <inertia
         ixx="64.8069935901443"
-        ixy="0.00212233959160378"
-        ixz="0.000377899491888311"
+        ixy="0.00212233959160385"
+        ixz="0.000377899491888313"
         iyy="42.2474032259228"
         iyz="-1.35082963675344"
@@ -557,5 +557,5 @@
     <inertial>
       <origin
-        xyz="7.22391839388936E-06 -0.000475137384490038 0.000654978643972126"
+        xyz="7.22391839388589E-06 -0.000475137384490121 0.000654978643972126"
         rpy="0 0 0" />
       <mass
@@ -563,8 +563,8 @@
       <inertia
         ixx="0.00312084570629235"
-        ixy="1.03835097415563E-07"
-        ixz="2.20016415043754E-07"
+        ixy="1.03835097415627E-07"
+        ixz="2.20016415043753E-07"
         iyy="0.00309492725703448"
-        iyz="5.55031448922626E-07"
+        iyz="5.55031448922631E-07"
         izz="0.00574920281992534" />
     </inertial>
@@ -610,15 +610,15 @@
     <inertial>
       <origin
-        xyz="3.70762208490617E-05 0.0114409852434533 0.0116125856420283"
-        rpy="0 0 0" />
-      <mass
-        value="8.30725875791486" />
-      <inertia
-        ixx="0.029020927491474"
-        ixy="7.55948089001623E-06"
-        ixz="-8.23045819536529E-06"
-        iyy="0.027224956518295"
-        iyz="0.00281819311295836"
-        izz="0.0270973700422314" />
+        xyz="3.70761457497565E-05 0.0114409856017593 0.0116125858663346"
+        rpy="0 0 0" />
+      <mass
+        value="8.30725872178856" />
+      <inertia
+        ixx="0.0290209274545541"
+        ixy="7.55947991125206E-06"
+        ixz="-8.23047846730788E-06"
+        iyy="0.0272249564707654"
+        iyz="0.00281819311419462"
+        izz="0.0270973700316767" />
     </inertial>
     <visual>
@@ -663,15 +663,15 @@
     <inertial>
       <origin
-        xyz="-2.43404147082064E-05 -0.250894715013332 -0.00563651299321782"
-        rpy="0 0 0" />
-      <mass
-        value="23.5085888532833" />
-      <inertia
-        ixx="0.256767671623099"
-        ixy="3.6239951788455E-06"
-        ixz="-9.72858775406846E-07"
-        iyy="0.0505710283974333"
-        iyz="0.00203684454830707"
-        izz="0.255664797838807" />
+        xyz="-2.43403882967536E-05 -0.250894715459623 -0.00563651311083996"
+        rpy="0 0 0" />
+      <mass
+        value="23.5085888172064" />
+      <inertia
+        ixx="0.256767671586333"
+        ixy="3.62397486865205E-06"
+        ixz="-9.72859790180711E-07"
+        iyy="0.0505710283867853"
+        iyz="0.00203684454960158"
+        izz="0.255664797791348" />
     </inertial>
     <visual>
@@ -716,14 +716,14 @@
     <inertial>
       <origin
-        xyz="0.244390991313135 -0.0139095256822837 -0.00101283060327786"
-        rpy="0 0 0" />
-      <mass
-        value="8.43948455874415" />
-      <inertia
-        ixx="0.00901829529744047"
-        ixy="-1.75583144369193E-06"
-        ixz="-0.00028822454084213"
+        xyz="-0.244390991313135 0.0139095256822855 -0.00101283060327773"
+        rpy="0 0 0" />
+      <mass
+        value="8.43948455874413" />
+      <inertia
+        ixx="0.00901829529744046"
+        ixy="-1.7558314428111E-06"
+        ixz="0.000288224540842122"
         iyy="0.131613662619847"
-        iyz="3.49342881189501E-07"
+        iyz="-3.49342881195927E-07"
         izz="0.131781826183782" />
     </inertial>
@@ -757,5 +757,5 @@
     <origin
       xyz="-0.014341662691355 -0.616041711362748 -0.127892362765015"
-      rpy="-3.14159265358979 0 -1.57079632679489" />
+      rpy="3.14159265358979 0 1.57079632679489" />
     <parent
       link="12" />
@@ -763,5 +763,5 @@
       link="23" />
     <axis
-      xyz="0 0.00340256352288005 0.999994211263982" />
+      xyz="0 -0.00340256352288005 0.999994211263982" />
   </joint>
   <link
@@ -769,15 +769,15 @@
     <inertial>
       <origin
-        xyz="-0.00758686877396642 -0.000158257963224488 0.00819784914576557"
-        rpy="0 0 0" />
-      <mass
-        value="0.728996428250046" />
-      <inertia
-        ixx="0.000910114210779735"
-        ixy="-4.95497562223844E-07"
-        ixz="-0.00012008521723334"
-        iyy="0.000986687923606722"
-        iyz="-1.62299300727913E-07"
-        izz="0.000877255272961634" />
+        xyz="0.00758686877396486 0.000158257963222184 0.0081978491457739"
+        rpy="0 0 0" />
+      <mass
+        value="0.728996428249931" />
+      <inertia
+        ixx="0.000910114210779709"
+        ixy="-4.95497562180507E-07"
+        ixz="0.000120085217233337"
+        iyy="0.000986687923606646"
+        iyz="1.62299300726255E-07"
+        izz="0.000877255272961533" />
     </inertial>
     <visual>
@@ -809,5 +809,5 @@
     type="continuous">
     <origin
-      xyz="0.568458717066326 -0.0140771361182816 -0.00154359819575967"
+      xyz="-0.568458717066326 0.0140771361182856 -0.00154359819575967"
       rpy="3.14159265358979 0 0" />
     <parent
@@ -816,5 +816,5 @@
       link="34" />
     <axis
-      xyz="-1 0 0" />
+      xyz="1 0 0" />
   </joint>
   <link
@@ -822,15 +822,15 @@
     <inertial>
       <origin
-        xyz="-6.86078064257925E-06 -0.00758686562123945 0.0107376301790445"
-        rpy="0 0 0" />
-      <mass
-        value="0.728996237064777" />
-      <inertia
-        ixx="0.000986687619429261"
-        ixy="-1.0315261819144E-09"
-        ixz="-4.1735472920583E-07"
-        iyy="0.000910112478523473"
-        iyz="-0.000120085251276709"
-        izz="0.000877253255884629" />
+        xyz="-6.86078063953655E-06 -0.00758686562124228 0.0107376301790323"
+        rpy="0 0 0" />
+      <mass
+        value="0.728996237064935" />
+      <inertia
+        ixx="0.000986687619429367"
+        ixy="-1.03152612309003E-09"
+        ixz="-4.1735472920365E-07"
+        iyy="0.000910112478523505"
+        iyz="-0.000120085251276714"
+        izz="0.000877253255884768" />
     </inertial>
     <visual>
@@ -862,6 +862,6 @@
     type="continuous">
     <origin
-      xyz="-0.00107999999999775 0.000121644413048502 0.114239846500137"
-      rpy="1.5707963267949 0 1.57079632679489" />
+      xyz="0.00107999999999753 -0.000121644413048495 0.114239846500137"
+      rpy="1.5707963267949 0 -1.57079632679489" />
     <parent
       link="34" />
@@ -875,15 +875,15 @@
     <inertial>
       <origin
-        xyz="-0.000158258378740259 0.00758689090859144 0.010737837609898"
-        rpy="0 0 0" />
-      <mass
-        value="0.728997478631908" />
-      <inertia
-        ixx="0.000986687250754589"
-        ixy="4.95491590354025E-07"
-        ixz="-1.62291043906281E-07"
-        iyy="0.000910112496687827"
-        iyz="0.000120084923500319"
-        izz="0.000877253430656248" />
+        xyz="-0.000158258378738691 0.00758689090859055 0.0107378376099037"
+        rpy="0 0 0" />
+      <mass
+        value="0.728997478631833" />
+      <inertia
+        ixx="0.00098668725075454"
+        ixy="4.9549159032517E-07"
+        ixz="-1.62291043904241E-07"
+        iyy="0.00091011249668781"
+        iyz="0.000120084923500316"
+        izz="0.000877253430656182" />
     </inertial>
     <visual>
@@ -928,5 +928,5 @@
     <inertial>
       <origin
-        xyz="-5.11211491377381E-05 -0.000470150585815121 -0.00309378276926542"
+        xyz="-5.11211491377346E-05 -0.000470150585814899 -0.00309378276926547"
         rpy="0 0 0" />
       <mass
@@ -981,5 +981,5 @@
     <inertial>
       <origin
-        xyz="-0.00710247160346223 0.0303390950483817 0.000488474590246035"
+        xyz="-0.00710247160346203 0.0303390950483818 0.000488474590246035"
         rpy="0 0 0" />
       <mass
@@ -987,8 +987,8 @@
       <inertia
         ixx="0.00651208089817064"
-        ixy="0.000182430404454022"
-        ixz="-0.000121865713788611"
-        iyy="0.00861283977900374"
-        iyz="-1.31090652690096E-05"
+        ixy="0.000182430404454018"
+        ixz="-0.00012186571378861"
+        iyy="0.00861283977900375"
+        iyz="-1.31090652690102E-05"
         izz="0.0049440363866004" />
     </inertial>
