Commit message: added vaccum gripper changed postion controller to accomidate vaccum gripper reduced linear velocity speed modified open loop controller to pause , go and stop

File: urdf/car.xacro (robot description, xacro)
@@ -1019,5 +1019,5 @@
   <joint
     name="7-gripper_joint"
-    type="fixed">
+    type="continuous">
     <origin
       xyz="-0.000514480216416438 0.000109109397764318 0.0968676227049757"
@@ -1117,4 +1117,12 @@
 </joint>
 <joint name="67j">
+  <command_interface name="velocity">
+      <param name="min">-1000.0</param>
+      <param name="max">1000.0</param>
+  </command_interface>
+  <state_interface name="position"/>
+  <state_interface name="velocity"/>
+</joint>
+<joint name="7-gripper_joint">
   <command_interface name="velocity">
       <param name="min">-1000.0</param>
@@ -1191,4 +1199,12 @@
 </joint>
 <joint name="67j">
+  <command_interface name="position">
+      <param name="min">-3.14</param>
+      <param name="max">3.14</param>
+  </command_interface>
+  <state_interface name="position"/>
+  <state_interface name="velocity"/>
+</joint>
+<joint name="7-gripper_joint">
   <command_interface name="position">
       <param name="min">-3.14</param>
@@ -1262,4 +1278,23 @@
         </plugin>
       </gazebo>
+      <gazebo>
+        <plugin name='vacuum_gripper' filename='libgazebo_ros_vacuum_gripper.so'>
+          <!-- This part can be commented out if not required -->
+          <ros>
+            <!-- Add a namespace -->
+            <namespace>/</namespace>
+            <!-- Remapping service and topic names -->
+            <remapping>switch:=custom_switch</remapping>
+            <remapping>grasping:=custom_grasping</remapping>
+          </ros>
+          <!-- Link associated with gripper -->
+          <link_name>gripper</link_name>
+          <!-- Max distance to attract entities -->
+          <max_distance>10.0</max_distance>
+          <!-- List of entities to be not attracted by the gripper -->
+          <fixed>ground_plane</fixed>
+          <fixed>wall</fixed>
+        </plugin>
+      </gazebo>
     <gazebo>
       <plugin filename="libgazebo_ros2_control.so" name="gazebo_ros2_control">
